Commit message: Split robot description into subassemblies using xacro

File: goldorak_description/urdf/goldorak.xacro (robot description, xacro)
@@ -10,22 +10,7 @@
   <xacro:property name="caster_radius" value="0.01" />
   <xacro:property name="caster_offset" value="-0.19" />
-  <xacro:property name="pi" value="3.1415" />
-  <material name="blue">
-    <color rgba="0 0 .8 1"/>
-  </material>
-  <material name="black">
-    <color rgba="0 0 0 1"/>
-  </material>
-  <material name="white">
-    <color rgba="1 1 1 1"/>
-  </material>
-  <xacro:macro name="default_inertial" params="mass">
-    <inertial>
-      <mass value="${mass}" />
-      <inertia ixx="1.0" ixy="0.0" ixz="0.0"
-               iyy="1.0" iyz="0.0"
-               izz="1.0" />
-    </inertial>
-  </xacro:macro>
+  <xacro:include filename="$(find goldorak_description)/urdf/common.urdf.xacro" />
+  <xacro:include filename="$(find goldorak_description)/urdf/wheel.urdf.xacro" />
+  <xacro:include filename="$(find goldorak_description)/urdf/caster.urdf.xacro" />
   <!-- Base link -->
   <link name="base_link">
@@ -49,106 +34,8 @@
     </inertial>
   </link>
-  <!-- Wheel link xacro -->
-  <xacro:macro name="wheel" params="prefix reflect">
-    <link name="${prefix}_wheel">
-      <visual>
-        <origin xyz="0 0 0" rpy="${pi/2} 0 0" />
-        <geometry>
-          <cylinder radius="${wheel_radius}" length="${wheel_thickness}"/>
-        </geometry>
-        <material name="black"/>
-        <origin xyz="0 0 0" rpy="0 0 0" />
-      </visual>
-      <collision>
-        <origin xyz="0 0 0" rpy="${pi/2} 0 0" />
-        <geometry>
-          <cylinder radius="${wheel_radius}" length="${wheel_thickness}"/>
-        </geometry>
-        <origin xyz="0 0 0" rpy="0 0 0" />
-      </collision>
-      <inertial>
-          <origin xyz="0 0 0"/>
-          <mass value="0.01" />
-          <inertia ixx="0.001" ixy="0.0" ixz="0.0"
-                   iyy="0.001" iyz="0.0"
-                   izz="0.001" />
-        </inertial>
-    </link>
-    <joint name="${prefix}_wheel_joint" type="continuous">
-      <axis xyz="0 1 0" rpy="0 0 0" />
-      <parent link="base_link"/>
-      <child link="${prefix}_wheel"/>
-      <origin xyz="0
-                   ${(wheelbase + wheel_thickness) * reflect / 2}
-                   ${wheel_offset - wheel_radius}"
-              rpy="0 0 0"/>
-    </joint>
-    <!-- This block provides the simulator (Gazebo) with information on a few additional
-    physical properties. See http://gazebosim.org/tutorials/?tut=ros_urdf for more-->
-    <gazebo reference="${prefix}_wheel">
-      <mu1>1.0</mu1>
-      <mu2>1.0</mu2>
-      <kp>1000000.0</kp>
-      <kd>100.0</kd>
-      <material>Gazebo/Grey</material>
-    </gazebo>
-    <!-- This block connects the wheel joint to an actuator (motor), which informs both
-    simulation and visualization of the robot -->
-    <transmission name="${prefix}_wheel_trans" type="SimpleTransmission">
-      <type>transmission_interface/SimpleTransmission</type>
-      <actuator name="${prefix}_wheel_motor">
-        <mechanicalReduction>1</mechanicalReduction>
-      </actuator>
-      <joint name="${prefix}_wheel_joint">
-        <hardwareInterface>VelocityJointInterface</hardwareInterface>
-      </joint>
-    </transmission>
-  </xacro:macro>
+  <!-- Wheels -->
   <xacro:wheel prefix="right" reflect="1"/>
   <xacro:wheel prefix="left" reflect="-1"/>
-  <xacro:macro name="caster" params="prefix reflect">
-    <link name="${prefix}_caster">
-      <visual>
-        <origin xyz="0 0 0" rpy="${pi/2} 0 0" />
-        <geometry>
-          <sphere radius="${caster_radius}" />
-        </geometry>
-        <material name="black"/>
-        <origin xyz="0 0 0" rpy="0 0 0" />
-      </visual>
-      <collision>
-        <origin xyz="0 0 0" rpy="${pi/2} 0 0" />
-        <geometry>
-          <sphere radius="${caster_radius}" />
-        </geometry>
-        <origin xyz="0 0 0" rpy="0 0 0" />
-      </collision>
-      <inertial>
-        <origin xyz="0 0 0" />
-        <mass value="0.01" />
-        <inertia ixx="0.001" ixy="0.0" ixz="0.0"
-                 iyy="0.001" iyz="0.0"
-                 izz="0.001" />
-        </inertial>
-    </link>
-    <joint name="${prefix}_caster_joint" type="fixed">
-      <axis xyz="0 1 0" rpy="0 0 0" />
-      <parent link="base_link"/>
-      <child link="${prefix}_caster"/>
-      <origin xyz="${(casterbase + caster_radius) * reflect / 2}
-                   0
-                   ${caster_offset - caster_radius}"
-              rpy="0 0 0"/>
-    </joint>
-    <gazebo reference="${prefix}_caster">
-      <mu1>0.0</mu1>
-      <mu2>0.0</mu2>
-      <kp>1000000.0</kp>
-      <kd>100.0</kd>
-      <minDepth>0.001</minDepth>
-      <maxVel>1.0</maxVel>
-      <material>Gazebo/Grey</material>
-    </gazebo>
-  </xacro:macro>
+  <!-- Casters -->
   <xacro:caster prefix="front" reflect="1"/>
   <xacro:caster prefix="rear" reflect="-1"/>

Commit message: Refactor laser sensor simulation into range sensor

File: goldorak_description/urdf/goldorak.xacro (robot description, xacro)
@@ -13,4 +13,5 @@
   <xacro:include filename="$(find goldorak_description)/urdf/wheel.urdf.xacro" />
   <xacro:include filename="$(find goldorak_description)/urdf/caster.urdf.xacro" />
+  <xacro:include filename="$(find goldorak_description)/urdf/range_sensor.urdf.xacro" />
   <!-- Base link -->
   <link name="base_link">
@@ -40,32 +41,4 @@
   <xacro:caster prefix="front" reflect="1"/>
   <xacro:caster prefix="rear" reflect="-1"/>
-  <!-- Laser scanner 1D link -->
-  <joint name="laser_joint" type="fixed">
-    <axis xyz="0 1 0" />
-    <origin xyz="0 0 ${body_height / 2}" rpy="0 0 0"/>
-    <parent link="base_link"/>
-    <child link="laser_link"/>
-  </joint>
-  <link name="laser_link">
-    <collision>
-      <origin xyz="0 0 0" rpy="0 0 0"/>
-      <geometry>
-        <cylinder radius="0.02" length="0.02"/>
-      </geometry>
-    </collision>
-    <visual>
-      <origin xyz="0 0 0" rpy="0 0 0"/>
-      <geometry>
-        <cylinder radius="0.02" length="0.02"/>
-      </geometry>
-    </visual>
-    <inertial>
-      <mass value="1e-5" />
-      <origin xyz="0 0 0" rpy="0 0 0"/>
-      <inertia ixx="1e-6" ixy="0" ixz="0"
-               iyy="1e-6" iyz="0"
-               izz="1e-6" />
-    </inertial>
-  </link>
   <!-- Gazebo plugin for ROS Control -->
   <gazebo>
@@ -74,35 +47,8 @@
     </plugin>
   </gazebo>
-  <!-- Gazebo plugin for Laser scanner -->
-  <gazebo reference="laser_link">
-    <sensor type="ray" name="laser_sensor">
-      <pose>0 0 0 0 0 0</pose>
-      <visualize>true</visualize>
-      <update_rate>40</update_rate>
-      <ray>
-        <scan>
-          <horizontal>
-            <samples>1</samples>
-            <resolution>1</resolution>
-            <min_angle>-1.570796</min_angle>
-            <max_angle>1.570796</max_angle>
-          </horizontal>
-        </scan>
-        <range>
-          <min>0.10</min>
-          <max>30.0</max>
-          <resolution>0.01</resolution>
-        </range>
-        <noise>
-          <type>gaussian</type>
-          <mean>0.0</mean>
-          <stddev>0.01</stddev>
-        </noise>
-      </ray>
-      <plugin name="gazebo_ros_laser_controller" filename="libgazebo_ros_laser.so">
-        <topicName>/laser/scan</topicName>
-        <frameName>laser_link</frameName>
-      </plugin>
-    </sensor>
-  </gazebo>
+  <!-- Laser scanner 1D link -->
+  <xacro:range_sensor name="laser" parent="base_link" rate="50"
+                      maxRange="4.0" minRange="0.15" fov="0.1">
+    <origin xyz="0 0 ${body_height / 2}" rpy="0 0 0"/>
+  </xacro:range_sensor>
 </robot>
